Commit message: perf: optimize omni wheel simulation model

File: khemin_omni/urdf/omni.urdf.xacro (robot description, xacro)
@@ -1,5 +1,4 @@
 <?xml version="1.0"?>
 <robot xmlns:xacro="http://ros.org/wiki/xacro">
-  <xacro:include filename="$(find khemin_omni)/urdf/roller.urdf.xacro"/>
   <xacro:macro name="omni_wheel" params="suffix parent xyz rpy">
     <link name="omni_wheel_link_${suffix}">
@@ -13,9 +12,10 @@
         </material>
       </visual>
-      <!-- <collision>
+      <collision>
+        <origin xyz="0 0 0" rpy="0 0 0"/>
         <geometry>
-          <mesh filename="package://khemin_omni/mesh/omni.stl" scale="0.001 0.001 0.001"/>
+          <cylinder radius="0.075" length="0.05"/>
         </geometry>
-      </collision> -->
+      </collision>
       <inertial>
         <mass value="0.5" />
@@ -30,20 +30,10 @@
       <axis xyz="0 0 -1"/>
     </joint>
-    <xacro:roller parent="omni_wheel_link_${suffix}" suffix="${suffix}1"  xyz="0.07 0 0.00175" rpy="-1.5708 0 3.1416"/>
-    <xacro:roller parent="omni_wheel_link_${suffix}" suffix="${suffix}2"  xyz="0.0647 0.0268 0.00175" rpy="-1.5708 0 3.5343"/>
-    <xacro:roller parent="omni_wheel_link_${suffix}" suffix="${suffix}3"  xyz="0.0495 0.0495 0.00175" rpy="-1.5708 0 3.9269"/>
-    <xacro:roller parent="omni_wheel_link_${suffix}" suffix="${suffix}4"  xyz="0.0268 0.0647 0.00175" rpy="-1.5708 0 4.3197"/>
-    <xacro:roller parent="omni_wheel_link_${suffix}" suffix="${suffix}5"  xyz="0 0.07 0.00175" rpy="-1.5708 0 4.7124"/>
-    <xacro:roller parent="omni_wheel_link_${suffix}" suffix="${suffix}6"  xyz="-0.0268 0.0647 0.00175" rpy="-1.5708 0 5.1051"/>
-    <xacro:roller parent="omni_wheel_link_${suffix}" suffix="${suffix}7"  xyz="-0.0495 0.0495 0.00175" rpy="-1.5708 0 5.4978"/>
-    <xacro:roller parent="omni_wheel_link_${suffix}" suffix="${suffix}8"  xyz="-0.0647 0.0268 0.00175" rpy="-1.5708 0 5.8905"/>
-    <xacro:roller parent="omni_wheel_link_${suffix}" suffix="${suffix}9"  xyz="-0.07 0 0.00175" rpy="-1.5708 0 0.0"/>
-    <xacro:roller parent="omni_wheel_link_${suffix}" suffix="${suffix}10" xyz="-0.0647 -0.0268 0.00175" rpy="-1.5708 0 0.3927"/>
-    <xacro:roller parent="omni_wheel_link_${suffix}" suffix="${suffix}11" xyz="-0.0495 -0.0495 0.00175" rpy="-1.5708 0 0.7854"/>
-    <xacro:roller parent="omni_wheel_link_${suffix}" suffix="${suffix}12" xyz="-0.0268 -0.0647 0.00175" rpy="-1.5708 0 1.1781"/>
-    <xacro:roller parent="omni_wheel_link_${suffix}" suffix="${suffix}13" xyz="0 -0.07 0.00175" rpy="-1.5708 0 1.5708"/>
-    <xacro:roller parent="omni_wheel_link_${suffix}" suffix="${suffix}14" xyz="0.0268 -0.0647 0.00175" rpy="-1.5708 0 1.9635"/>
-    <xacro:roller parent="omni_wheel_link_${suffix}" suffix="${suffix}15" xyz="0.0495 -0.0495 0.00175" rpy="-1.5708 0 2.3562"/>
-    <xacro:roller parent="omni_wheel_link_${suffix}" suffix="${suffix}16" xyz="0.0647 -0.0268 0.00175" rpy="-1.5708 0 2.7489"/>
+    <gazebo reference="omni_wheel_link_${suffix}">
+      <selfCollide>false</selfCollide>
+      <mu1>1.0</mu1>
+      <mu2>0.001</mu2>
+      <fdir1>1 0 0</fdir1>
+    </gazebo>
   </xacro:macro>
 </robot>
